Commit message: Added some visualization launch files for the franka

File: aloha4franka_description/urdf/aloha_gripper_base.urdf.xacro (robot description, xacro)
@@ -1,6 +1,7 @@
 <?xml version="1.0" ?>
 <robot name="aloha_gripper" xmlns:xacro="http://ros.org/wiki/xacro">
-   <xacro:macro name="aloha_gripper_base" params="parent">
+   <xacro:macro name="aloha_gripper_base" params="parent *origin">
       <joint name="parent_to_attachment" type="fixed">
+         <xacro:insert_block name="origin" />
          <parent link="${parent}" />
          <child link="attachment" />
