Commit message: Modified values for real gripper + added media

File: aloha4franka_description/urdf/aloha_gripper.ros2_control.urdf.xacro (robot description, xacro)
@@ -6,6 +6,6 @@
         <plugin>dynamixel_hardware/DynamixelHardware</plugin>
         <param name="usb_port">/dev/ttyUSB0</param>
-        <param name="baud_rate">1000000</param>
-        <param name="use_dummy">true</param>
+        <param name="baud_rate">57600</param>
+        <param name="use_dummy">false</param>
       </hardware>
       <joint name="left_finger_joint">
@@ -17,4 +17,12 @@
         <state_interface name="effort"/>
       </joint>
+      <transmission name="transmission1">
+        <plugin>transmission_interface/SimpleTransmission</plugin>
+        <actuator name="actuator" role="actuator"/>
+        <joint name="left_finger_joint" role="left_finger_joint">
+          <mechanical_reduction>100.0</mechanical_reduction>
+          <offset>0.0</offset>
+        </joint>
+      </transmission>
     </ros2_control>
   </xacro:macro>

File: aloha4franka_description/urdf/aloha_gripper.urdf.xacro (robot description, xacro)
@@ -4,5 +4,7 @@
   <xacro:include filename="$(find aloha4franka_description)/urdf/aloha_gripper.ros2_control.urdf.xacro" />
   <link name="world"/>
-  <xacro:aloha_gripper_base parent="world"/>
-  <xacro:aloha_gripper_ros2_control name="aloha_gripper_ros2_control" use_dummy="true"/>
+  <xacro:aloha_gripper_base parent="world">
+    <origin xyz="0 0 0" rpy="0 0 -3.7524578918" />
+  </xacro:aloha_gripper_base>
+  <xacro:aloha_gripper_ros2_control name="aloha_gripper_ros2_control" use_dummy="false"/>
 </robot>

Commit message: Allow uncontrolled motor (only temporary, soon chaning to different package)

File: aloha4franka_description/urdf/aloha_gripper.ros2_control.urdf.xacro (robot description, xacro)
@@ -1,9 +1,9 @@
 <?xml version="1.0"?>
 <robot xmlns:xacro="http://www.ros.org/wiki/xacro">
-  <xacro:macro name="aloha_gripper_ros2_control" params="name use_dummy">
+  <xacro:macro name="aloha_gripper_ros2_control" params="name use_dummy device uncontrolled">
     <ros2_control name="${name}" type="system">
       <hardware>
         <plugin>dynamixel_hardware/DynamixelHardware</plugin>
-        <param name="usb_port">/dev/ttyUSB0</param>
+        <param name="usb_port">${device}</param>
         <param name="baud_rate">57600</param>
         <param name="use_dummy">false</param>
@@ -11,4 +11,11 @@
       <joint name="left_finger_joint">
         <param name="id">1</param>
+      <xacro:if value="${uncontrolled}">
+        <param name="Position_P_Gain">0</param>
+        <param name="Position_I_Gain">0</param>
+        <param name="Position_D_Gain">0</param>
+        <param name="Velocity_P_Gain">0</param>
+        <param name="Velocity_I_Gain">0</param>
+      </xacro:if>
         <command_interface name="position"/>
         <command_interface name="velocity"/>

File: aloha4franka_description/urdf/aloha_gripper.urdf.xacro (robot description, xacro)
@@ -3,8 +3,11 @@
   <xacro:include filename="$(find aloha4franka_description)/urdf/aloha_gripper_base.urdf.xacro" />
   <xacro:include filename="$(find aloha4franka_description)/urdf/aloha_gripper.ros2_control.urdf.xacro" />
+  <!--<xacro:arg name="use_dummy" default="false" />-->
+  <xacro:arg name="device" default="/dev/ttyUSB0" />
+  <xacro:arg name="uncontrolled" default="false" />
   <link name="world"/>
   <xacro:aloha_gripper_base parent="world">
     <origin xyz="0 0 0" rpy="0 0 -3.7524578918" />
   </xacro:aloha_gripper_base>
-  <xacro:aloha_gripper_ros2_control name="aloha_gripper_ros2_control" use_dummy="false"/>
+  <xacro:aloha_gripper_ros2_control name="aloha_gripper_ros2_control" use_dummy="false" device="$(arg device)" uncontrolled="$(arg uncontrolled)"/>
 </robot>

Commit message: udev rules, param description, new gripper backend

File: aloha4franka_description/urdf/aloha_gripper.ros2_control.urdf.xacro (robot description, xacro)
@@ -4,32 +4,44 @@
     <ros2_control name="${name}" type="system">
       <hardware>
-        <plugin>dynamixel_hardware/DynamixelHardware</plugin>
-        <param name="usb_port">${device}</param>
-        <param name="baud_rate">57600</param>
-        <param name="use_dummy">false</param>
+          <plugin>dynamixel_hardware_interface/DynamixelHardware</plugin>
+          <param name="port_name">${device}</param>
+          <param name="baud_rate">57600</param>
+          <param name="error_timeout_ms">100</param>
+          <param name="dynamixel_model_folder">/param/dxl_model</param>
+          <param name="number_of_joints">1</param>
+          <param name="number_of_transmissions">1</param>
+          <param name="transmission_to_joint_matrix">1</param>
+          <param name="joint_to_transmission_matrix">1</param>
+          <param name="dynamixel_state_pub_msg_name">dynamixel_hardware_interface/dxl_state</param>
+          <param name="get_dynamixel_data_srv_name">dynamixel_hardware_interface/get_dxl_data</param>
+          <param name="set_dynamixel_data_srv_name">dynamixel_hardware_interface/set_dxl_data</param>
+          <param name="reboot_dxl_srv_name">dynamixel_hardware_interface/reboot_dxl</param>
+          <param name="set_dxl_torque_srv_name">dynamixel_hardware_interface/set_dxl_torque</param>
+          <!-- This parameter is used for a prismatic joint that operates through a revolute mechanism.
+          If the joint does not require this configuration, this parameter can be removed. -->
+          <!--<param name="use_revolute_to_prismatic_gripper">1</param>-->
+          <!--<param name="revolute_to_prismatic_dxl">dxl</param>-->
+          <!--<param name="revolute_max">1.51</param>-->
+          <!--<param name="revolute_min">0.56</param>-->
+          <!--<param name="revolute_to_prismatic_joint">left_finger_joint</param>-->
+          <!--<param name="prismatic_max">0.019</param>-->
+          <!--<param name="prismatic_min">-0.01</param>-->
       </hardware>
       <joint name="left_finger_joint">
         <param name="id">1</param>
-      <xacro:if value="${uncontrolled}">
-        <param name="Position_P_Gain">0</param>
-        <param name="Position_I_Gain">0</param>
-        <param name="Position_D_Gain">0</param>
-        <param name="Velocity_P_Gain">0</param>
-        <param name="Velocity_I_Gain">0</param>
-      </xacro:if>
         <command_interface name="position"/>
-        <command_interface name="velocity"/>
+        <!--<command_interface name="effort"/>-->
         <state_interface name="position"/>
         <state_interface name="velocity"/>
         <state_interface name="effort"/>
       </joint>
-      <transmission name="transmission1">
-        <plugin>transmission_interface/SimpleTransmission</plugin>
-        <actuator name="actuator" role="actuator"/>
-        <joint name="left_finger_joint" role="left_finger_joint">
-          <mechanical_reduction>100.0</mechanical_reduction>
-          <offset>0.0</offset>
-        </joint>
-      </transmission>
+      <gpio name="dxl1">
+        <param name="type">dxl</param>
+        <param name="ID">1</param>
+        <command_interface name="Goal Position"/>
+        <state_interface name="Present Position"/>
+        <state_interface name="Present Velocity"/>
+        <state_interface name="Present Load"/>
+      </gpio>
     </ros2_control>
   </xacro:macro>

File: aloha4franka_description/urdf/aloha_gripper_base.urdf.xacro (robot description, xacro)
@@ -157,5 +157,5 @@
          <axis xyz="0 0 -1"/>
          <mimic joint="left_finger_joint" multiplier="1.0" offset="0.0"/>
-         <limit lower="0.0" upper="0.041" effort="20" velocity="0.1"/>
+         <limit lower="-100.0" upper="100.0" effort="20" velocity="0.1"/>
       </joint>
       <joint type="fixed" name="right_finger_offset">

Commit message: Added a lot of functions for daignostic publishing

File: aloha4franka_description/urdf/aloha_gripper.ros2_control.urdf.xacro (robot description, xacro)
@@ -7,4 +7,5 @@
           <param name="port_name">${device}</param>
           <param name="baud_rate">57600</param>
+          <param name="disable_torque_at_init">true</param>
           <param name="error_timeout_ms">100</param>
           <param name="dynamixel_model_folder">/param/dxl_model</param>
@@ -31,5 +32,6 @@
         <param name="id">1</param>
         <command_interface name="position"/>
-        <!--<command_interface name="effort"/>-->
+        <command_interface name="velocity"/>
+        <command_interface name="effort"/>
         <state_interface name="position"/>
         <state_interface name="velocity"/>
@@ -40,7 +42,12 @@
         <param name="ID">1</param>
         <command_interface name="Goal Position"/>
+        <command_interface name="Goal Velocity"/>
+        <command_interface name="Goal PWM"/>
         <state_interface name="Present Position"/>
         <state_interface name="Present Velocity"/>
         <state_interface name="Present Load"/>
+        <param name="Drive Mode">0</param>
+        <param name="Operating Mode">3</param>
+        <param name="Return Delay Time">0</param>
       </gpio>
     </ros2_control>

File: aloha4franka_description/urdf/aloha_trigger.ros2_control.urdf.xacro (robot description, xacro)
@@ -1,5 +1,5 @@
 <?xml version="1.0"?>
 <robot xmlns:xacro="http://www.ros.org/wiki/xacro">
-  <xacro:macro name="aloha_trigger_and_gripper_ros2_control" params="name use_dummy device">
+  <xacro:macro name="aloha_trigger_ros2_control" params="name use_dummy device">
     <ros2_control name="${name}" type="system">
       <hardware>
@@ -9,14 +9,8 @@
           <!--<param name="error_timeout_ms">100</param>-->
           <param name="dynamixel_model_folder">/param/dxl_model</param>
-          <param name="number_of_joints">2</param>
-          <param name="number_of_transmissions">2</param>
-          <param name="transmission_to_joint_matrix">
-            1, 0,
-            0, 1
-          </param>
-          <param name="joint_to_transmission_matrix">
-            1, 0,
-            0, 1
-          </param>
+          <param name="number_of_joints">1</param>
+          <param name="number_of_transmissions">1</param>
+          <param name="transmission_to_joint_matrix">1</param>
+          <param name="joint_to_transmission_matrix">1</param>
           <param name="dynamixel_state_pub_msg_name">dynamixel_hardware_interface/dxl_state</param>
           <param name="get_dynamixel_data_srv_name">dynamixel_hardware_interface/get_dxl_data</param>
@@ -34,34 +28,9 @@
           <!--<param name="prismatic_min">-0.01</param>-->
       </hardware>
-      <joint name="left_finger_joint">
-        <param name="id">1</param>
-        <command_interface name="position"/>
-        <!--<command_interface name="velocity"/>-->
-        <!--<command_interface name="effort"/>-->
-        <state_interface name="position"/>
-        <state_interface name="velocity"/>
-        <!--<state_interface name="effort"/>-->
-      </joint>
-      <gpio name="dxl1">
-        <param name="type">dxl</param>
-        <param name="ID">1</param>
-        <command_interface name="Goal Position"/>
-        <!--<command_interface name="Goal Velocity"/>-->
-        <!--<command_interface name="Goal PWM"/>-->
-        <state_interface name="Present Position"/>
-        <state_interface name="Present Velocity"/>
-        <!--<state_interface name="Present Load"/>-->
-        <param name="Position P Gain">100</param> <!-- Proportional gain for position control -->
-        <param name="Position I Gain">0</param> <!-- Integral gain for position control -->
-        <param name="Position D Gain">0</param> <!-- Derivative gain for position control -->
-        <param name="Drive Mode">0</param>
-        <param name="Operating Mode">3</param>
-        <param name="Return Delay Time">0</param>
-      </gpio>
       <joint name="trigger_joint">
         <command_interface name="effort"/>
         <state_interface name="position"/>
         <state_interface name="velocity"/>
-        <!--<state_interface name="effort"/>-->
+        <state_interface name="effort"/>
       </joint>
       <gpio name="dxl2">
@@ -71,5 +40,5 @@
         <state_interface name="Present Position"/>
         <state_interface name="Present Velocity"/>
-        <!--<state_interface name="Present Load"/>-->
+        <state_interface name="Present Load"/>
         <param name="Drive Mode">0</param>
         <param name="Operating Mode">16</param>

File: aloha4franka_description/urdf/aloha_trigger_and_gripper.urdf.xacro (robot description, xacro)
@@ -1,8 +1,8 @@
 <?xml version="1.0"?>
 <robot name="aloha_gripper" xmlns:xacro="http://ros.org/wiki/xacro">
+  <xacro:include filename="$(find aloha4franka_description)/urdf/aloha_gripper_base.urdf.xacro" />
   <xacro:include filename="$(find aloha4franka_description)/urdf/aloha_trigger_and_gripper.ros2_control.urdf.xacro" />
   <!--<xacro:arg name="use_dummy" default="false" />-->
   <xacro:arg name="device" default="/dev/ttyUSB0" />
-  <xacro:arg name="uncontrolled" default="false" />
   <link name="world"/>
   <xacro:aloha_gripper_base parent="world">
@@ -13,5 +13,6 @@
       <parent link="gripper_base"/>
       <child link="trigger_link"/>
+      <limit lower="0.0" upper="0.5" effort="20" velocity="0.1"/>
   </joint>
-  <xacro:aloha_trigger_and_gripper_ros2_control name="aloha_trigger_and_gripper_ros2_control" use_dummy="false" device="$(arg device)" uncontrolled="$(arg uncontrolled)"/>
+  <xacro:aloha_trigger_and_gripper_ros2_control name="aloha_trigger_and_gripper_ros2_control" use_dummy="false" device="$(arg device)"/>
 </robot>
